File: hardware/board/Instability_VCA.kicad_sch (KiCad schematic)
At the start: 42 parts

Commit message: Rough Draft of Routing Complete. Ugly but Passes DRC
Parts:
- removed D?: BAS315, winterbloom:D_SOD-323, symbol Diode:1N5819
- added D?: BAS315, winterbloom:D_SOD-323, symbol Device:D_Small
Connections:
- net -8VREF: now also D?.2 (A)
- net at R?.1, R?.2: now also D?.1 (K)
Other:
- note added: "Controls the depth of the Instability feedback circuit Rectifies, AC Couples, and Clips filter output before using it to modulate Cutoff Frequency CV input: 5v Nominal Max Instability In High Pass Cutoff Frequency: TBD Instability In Low Pass Cutoff Frequency: TBD CV Cutoff: ~2.5khz"
- note added: "Input Filtering can be adjusted to tune the instability I couldn't make up my mind about which instability circuit to use, so I added solder jumpers so we can choose between them on the prototype."
- note removed: "Controls the depth of the Instability feedback circuit Rectifies, AC Couples, and Clips filter output before using it to modulate Cutoff Frequency CV input: 5v Nominal Max Instability In High Pass Cutoff Frequency: TBD Instability In Low Pass Cutoff Frequency: TBD CV Cutoff: ~2.5khz LED Max Brightness: 3.3mA"
- note removed: "Input Filtering can be adjusted to tune the instability I couldn't make up my mind about which instability circuit to use, so I added solder jumpers so we can choose between them on the prototype. Buffer after rectifier can probably be removed if we need to save an op amp"
Changed lines of the file:
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@@
+    (stroke (width 0) (type default))
+  )
+  (wire (pts (xy 135.89 151.13) (xy 135.89 152.4))
     (stroke (width 0) (type default))
   )
@@
     (stroke (width 0) (type default))
   )
-  (wire (pts (xy 135.89 140.97) (xy 135.89 144.78))
+  (wire (pts (xy 135.89 140.97) (xy 135.89 146.05))
     (stroke (width 0) (type default))
   )
@@
     (effects (font (size 5 5) (thickness 0.508) bold) (justify left bottom))
   )
-  (text "Controls the depth of the Instability feedback circuit\nRectifies, AC Couples, and Clips filter output before using it to modulate Cutoff Frequency\n\nCV input: 5v Nominal Max\n\nInstability In High Pass Cutoff Frequency: TBD\n\nInstability In Low Pass Cutoff Frequency: TBD\n\nCV Cutoff: ~2.5khz\n\nLED Max Brightness: 3.3mA\n"
-    (at 24.13 54.61 0)
+  (text "Controls the depth of the Instability feedback circuit\nRectifies, AC Couples, and Clips filter output before using it to modulate Cutoff Frequency\n\nCV input: 5v Nominal Max\n\nInstability In High Pass Cutoff Frequency: TBD\n\nInstability In Low Pass Cutoff Frequency: TBD\n\nCV Cutoff: ~2.5khz\n"
+    (at 24.13 50.8 0)
     (effects (font (size 1.27 1.27)) (justify left bottom))
   )
-  (text "Input Filtering can be adjusted to tune the instability \n\nI couldn't make up my mind about which instability circuit to use,\nso I added solder jumpers so we can choose between them on the prototype.\n\nBuffer after rectifier can probably be removed if we need to save an op amp\n"
-    (at 175.26 44.45 0)
+  (text "Input Filtering can be adjusted to tune the instability \n\nI couldn't make up my mind about which instability circuit to use,\nso I added solder jumpers so we can choose between them on the prototype."
+    (at 175.895 40.64 0)
     (effects (font (size 1.27 1.27)) (justify left bottom))
   )
@@
     )
   )
+  (symbol (lib_id "Device:D_Small") (at 135.89 148.59 90) (mirror x) (unit 1)
+    (in_bom yes) (on_board yes) (dnp no)
+    (property "Reference" "D?" (at 144.145 146.05 90)
+      (effects (font (size 1.27 1.27)))
+    )
+    (property "Value" "BAS315" (at 144.145 148.59 90)
+      (effects (font (size 1.27 1.27)))
+    )
+    (property "Footprint" "winterbloom:D_SOD-323" (at 135.89 148.59 90)
+      (effects (font (size 1.27 1.27)) hide)
+    )
+    (property "Datasheet" "~" (at 135.89 148.59 90)
+      (effects (font (size 1.27 1.27)) hide)
+    )
+    (property "MPN" "BAS316,115" (at 135.89 148.59 0)
+      (effects (font (size 1.27 1.27)) hide)
+    )
+    (property "Rating" "1Vf @ 100mA" (at 144.145 151.13 90)
+      (effects (font (size 1.27 1.27)))
+    )
+    (property "Notes" "Clipping diode" (at 135.89 148.59 0)
+      (effects (font (size 1.27 1.27)) hide)
+    )
+    (pin "1")
+    (pin "2")
+    (instances
+      (project "mainboard"
+        (path "/960bd036-bf0c-45ea-9f41-1321756e0e5a"
+          (reference "D?") (unit 1)
+        )
+        (path "/960bd036-bf0c-45ea-9f41-1321756e0e5a/3b1fa3f2-493c-449c-a2d6-10ea677680a0"
+          (reference "D?") (unit 1)
+        )
+        (path "/960bd036-bf0c-45ea-9f41-1321756e0e5a/48d891c0-35ba-4c8e-a930-c990a10298eb"
+          (reference "D?") (unit 1)
+        )
+        (path "/960bd036-bf0c-45ea-9f41-1321756e0e5a/0f8a3c3e-e197-47b5-881d-2ae4e2374020"
+          (reference "D702") (unit 1)
+        )
+      )
+      (project "Diode_Ladder_Filter_V0.5"
+        (path "/e63e39d7-6ac0-4ffd-8aa3-1841a4541b55"
+          (reference "D?") (unit 1)
+        )
+      )
+    )
+  )
   (symbol (lib_id "power:GND") (at 236.22 152.4 0) (unit 1)
     (in_bom yes) (on_board yes) (dnp no) (fields_autoplaced)
@@
   (symbol (lib_id "Device:D_Small") (at 107.95 82.55 0) (mirror y) (unit 1)
     (in_bom yes) (on_board yes) (dnp no)
-    (property "Reference" "D?" (at 107.95 73.66 0)
-      (effects (font (size 1.27 1.27)))
-    )
-    (property "Value" "BAS315" (at 107.95 76.2 0)
+    (property "Reference" "D?" (at 117.475 80.01 0)
+      (effects (font (size 1.27 1.27)))
+    )
+    (property "Value" "BAS315" (at 117.475 82.55 0)
       (effects (font (size 1.27 1.27)))
     )
@@
       (effects (font (size 1.27 1.27)) hide)
     )
-    (property "Rating" "1Vf @ 100mA" (at 107.95 78.74 0)
+    (property "Rating" "1Vf @ 100mA" (at 117.475 85.09 0)
       (effects (font (size 1.27 1.27)))
     )
@@
         )
       )
-    )
-  )
-  (symbol (lib_id "Diode:1N5819") (at 135.89 148.59 270) (unit 1)
-    (in_bom yes) (on_board yes) (dnp no)
-    (property "Reference" "D?" (at 138.43 146.3675 90)
-      (effects (font (size 1.27 1.27)) (justify left))
-    )
-    (property "Value" "BAS315" (at 138.43 148.9075 90)
-      (effects (font (size 1.27 1.27)) (justify left))
-    )
-    (property "Footprint" "winterbloom:D_SOD-323" (at 131.445 148.59 0)
-      (effects (font (size 1.27 1.27)) hide)
-    )
-    (property "Datasheet" "http://www.vishay.com/docs/88525/1n5817.pdf" (at 135.89 148.59 0)
-      (effects (font (size 1.27 1.27)) hide)
-    )
-    (property "Notes" "Clipping diode" (at 135.89 148.59 0)
-      (effects (font (size 1.27 1.27)) hide)
-    )
-    (property "Rating" "1Vf @ 100mA" (at 138.43 151.4475 90)
-      (effects (font (size 1.27 1.27)) (justify left))
-    )
-    (property "MPN" "BAS316,115" (at 135.89 148.59 0)
-      (effects (font (size 1.27 1.27)) hide)
-    )
-    (pin "1")
-    (pin "2")
-    (instances
-      (project "board"
-        (path "/55082cc1-c956-45a6-b2b5-3db02a6da9d0"
-          (reference "D?") (unit 1)
-        )
-      )
-      (project "mainboard"
-        (path "/960bd036-bf0c-45ea-9f41-1321756e0e5a/48d891c0-35ba-4c8e-a930-c990a10298eb"
-          (reference "D?") (unit 1)
-        )
-        (path "/960bd036-bf0c-45ea-9f41-1321756e0e5a/0f8a3c3e-e197-47b5-881d-2ae4e2374020"
-          (reference "D702") (unit 1)
-        )
-      )
-      (project "VCA"
-        (path "/de69ad6f-07bb-4f9c-962b-520f6532317d"
-          (reference "D?") (unit 1)
-        )
-        (path "/de69ad6f-07bb-4f9c-962b-520f6532317d/0f818280-e6cd-4382-a215-72bb59f50cc3"
-          (reference "D?") (unit 1)
-        )
-      )

Commit message: Final touches before being ready for ordering
Connections:
- net at U?.7: now also D?.1 (K); no longer D?.2 (A)
- net at JP702.2 (B), R?.1: now also D?.2 (A); no longer D?.1 (K)
Changed lines of the file:
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@@
     )
   )
-  (symbol (lib_id "Device:D_Small") (at 107.95 82.55 0) (mirror y) (unit 1)
+  (symbol (lib_id "Device:D_Small") (at 107.95 82.55 0) (unit 1)
     (in_bom yes) (on_board yes) (dnp no)
-    (property "Reference" "D?" (at 117.475 80.01 0)
+    (property "Reference" "D?" (at 116.84 80.01 0)
       (effects (font (size 1.27 1.27)))
     )
-    (property "Value" "BAS315" (at 117.475 82.55 0)
+    (property "Value" "BAS315" (at 116.84 82.55 0)
       (effects (font (size 1.27 1.27)))
     )
@@
       (effects (font (size 1.27 1.27)) hide)
     )
-    (property "Rating" "1Vf @ 100mA" (at 117.475 85.09 0)
+    (property "Rating" "1Vf @ 100mA" (at 116.84 85.09 0)
       (effects (font (size 1.27 1.27)))
     )
