File: hardware/board/Resonance_VCA.kicad_sch (KiCad schematic)
At the start: 31 parts

Commit message: Rough Draft of Routing Complete. Ugly but Passes DRC
Parts:
- removed D?: BAS315, winterbloom:D_SOD-323, symbol Diode:1N5819
- added D?: BAS315, winterbloom:D_SOD-323, symbol Device:D_Small
Connections:
- net -8VREF: now also D?.2 (A)
- net at R?.1, R?.2: now also D?.1 (K)
Other:
- note added: "Controls the depth of the Resonance feedback circuit CV input: 5V Nominal Max Self Resonance Gain Threshold: -8dB CV Cutoff: ~2.5khz Max Gain: -5.5dB Max Self Resonant Frequency: ~3kHz"
- note removed: "Controls the depth of the Resonance feedback circuit CV input: 5V Nominal Max Self Resonance Gain Threshold: -8dB CV Cutoff: ~2.5khz Max Gain: -5.5dB Max Self Resonant Frequency: ~3kHz LED Max Brightness: 4mA"
Changed lines of the file:
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@@
+    (stroke (width 0) (type default))
+  )
+  (wire (pts (xy 156.21 121.92) (xy 156.21 124.46))
     (stroke (width 0) (type default))
   )
@@
     (effects (font (size 5 5) (thickness 0.508) bold) (justify left bottom))
   )
-  (text "Controls the depth of the Resonance feedback circuit \n\nCV input: 5V Nominal Max\n\nSelf Resonance Gain Threshold: -8dB\n\nCV Cutoff: ~2.5khz\n\nMax Gain: -5.5dB\n\nMax Self Resonant Frequency: ~3kHz\n\nLED Max Brightness: 4mA\n\n\n"
-    (at 20.32 58.42 0)
+  (text "Controls the depth of the Resonance feedback circuit \n\nCV input: 5V Nominal Max\n\nSelf Resonance Gain Threshold: -8dB\n\nCV Cutoff: ~2.5khz\n\nMax Gain: -5.5dB\n\nMax Self Resonant Frequency: ~3kHz\n\n\n"
+    (at 20.32 55.245 0)
     (effects (font (size 1.27 1.27)) (justify left bottom))
   )
@@
     )
   )
-  (symbol (lib_id "Diode:1N5819") (at 156.21 120.65 270) (unit 1)
-    (in_bom yes) (on_board yes) (dnp no) (fields_autoplaced)
-    (property "Reference" "D?" (at 158.75 118.4275 90)
-      (effects (font (size 1.27 1.27)) (justify left))
-    )
-    (property "Value" "BAS315" (at 158.75 120.9675 90)
-      (effects (font (size 1.27 1.27)) (justify left))
-    )
-    (property "Footprint" "winterbloom:D_SOD-323" (at 151.765 120.65 0)
-      (effects (font (size 1.27 1.27)) hide)
-    )
-    (property "Datasheet" "http://www.vishay.com/docs/88525/1n5817.pdf" (at 156.21 120.65 0)
-      (effects (font (size 1.27 1.27)) hide)
-    )
-    (property "Notes" "Clipping diode" (at 156.21 120.65 0)
-      (effects (font (size 1.27 1.27)) hide)
-    )
-    (property "Rating" "1Vf @ 100mA" (at 158.75 123.5075 90)
-      (effects (font (size 1.27 1.27)) (justify left))
-    )
-    (property "MPN" "BAS316,115" (at 156.21 120.65 0)
-      (effects (font (size 1.27 1.27)) hide)
-    )
-    (pin "1")
-    (pin "2")
-    (instances
-      (project "board"
-        (path "/55082cc1-c956-45a6-b2b5-3db02a6da9d0"
-          (reference "D?") (unit 1)
-        )
-      )
-      (project "mainboard"
-        (path "/960bd036-bf0c-45ea-9f41-1321756e0e5a/48d891c0-35ba-4c8e-a930-c990a10298eb"
-          (reference "D601") (unit 1)
-        )
-      )
-      (project "VCA"
-        (path "/de69ad6f-07bb-4f9c-962b-520f6532317d"
-          (reference "D?") (unit 1)
-        )
-        (path "/de69ad6f-07bb-4f9c-962b-520f6532317d/0f818280-e6cd-4382-a215-72bb59f50cc3"
-          (reference "D?") (unit 1)
-        )
-      )
-    )
-  )
   (symbol (lib_id "power:GND") (at 218.44 127 0) (unit 1)
     (in_bom yes) (on_board yes) (dnp no) (fields_autoplaced)
@@
         )
       )
+    )
+  )
+  (symbol (lib_id "Device:D_Small") (at 156.21 119.38 90) (mirror x) (unit 1)
+    (in_bom yes) (on_board yes) (dnp no)
+    (property "Reference" "D?" (at 165.735 116.84 90)
+      (effects (font (size 1.27 1.27)))
+    )
+    (property "Value" "BAS315" (at 165.735 119.38 90)
+      (effects (font (size 1.27 1.27)))
+    )
+    (property "Footprint" "winterbloom:D_SOD-323" (at 156.21 119.38 90)
+      (effects (font (size 1.27 1.27)) hide)
+    )
+    (property "Datasheet" "~" (at 156.21 119.38 90)
+      (effects (font (size 1.27 1.27)) hide)
+    )
+    (property "MPN" "BAS316,115" (at 156.21 119.38 0)
+      (effects (font (size 1.27 1.27)) hide)
+    )
+    (property "Rating" "1Vf @ 100mA" (at 165.735 121.92 90)
+      (effects (font (size 1.27 1.27)))
+    )
+    (property "Notes" "Clipping diode" (at 156.21 119.38 0)
+      (effects (font (size 1.27 1.27)) hide)
+    )
+    (pin "1")
+    (pin "2")
+    (instances
+      (project "mainboard"
+        (path "/960bd036-bf0c-45ea-9f41-1321756e0e5a"
+          (reference "D?") (unit 1)
+        )
+        (path "/960bd036-bf0c-45ea-9f41-1321756e0e5a/3b1fa3f2-493c-449c-a2d6-10ea677680a0"
+          (reference "D?") (unit 1)
+        )
+        (path "/960bd036-bf0c-45ea-9f41-1321756e0e5a/48d891c0-35ba-4c8e-a930-c990a10298eb"
+          (reference "D601") (unit 1)
+        )
+        (path "/960bd036-bf0c-45ea-9f41-1321756e0e5a/0f8a3c3e-e197-47b5-881d-2ae4e2374020"
+          (reference "D701") (unit 1)
+        )
+      )
+      (project "Diode_Ladder_Filter_V0.5"
+        (path "/e63e39d7-6ac0-4ffd-8aa3-1841a4541b55"
+          (reference "D?") (unit 1)
+        )
+      )

Commit message: hardware: minor fixes and aesthetic updates
- Fix HP LEDs being backwards
- Switch power header, pot, and jack footprints to longpad variants
- Make the text size on the front side larger
- Add "red" and "blue" text next to respective LEDs on front side
- Adjusted zone thermal spoke for better connection to GND pads
- Squished the solder jumpers for instability type closer together
- Minor adjustments to traces to accommodate longpad footprints
Parts:
- J?: footprint winterbloom:AudioJack_WQP518MA_Compact_S -> winterbloom:AudioJack_WQP518MA_Compact_S_LongPads
- RV?: footprint winterbloom:Potentiometer_Alpha_R0904N -> winterbloom:Potentiometer_Alpha_R0904N_LongPads
Changed lines of the file:
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@@
       (effects (font (size 1.27 1.27)))
     )
-    (property "Footprint" "winterbloom:AudioJack_WQP518MA_Compact_S" (at 26.67 77.47 0)
+    (property "Footprint" "winterbloom:AudioJack_WQP518MA_Compact_S_LongPads" (at 26.67 77.47 0)
       (effects (font (size 1.27 1.27)) hide)
     )
@@
       (effects (font (size 1.27 1.27)) (justify left))
     )
-    (property "Footprint" "winterbloom:Potentiometer_Alpha_R0904N" (at 59.69 138.43 0)
-      (effects (font (size 1.27 1.27)) hide)
-    )
+    (property "Footprint" "winterbloom:Potentiometer_Alpha_R0904N_LongPads" (at 59.69 138.43 0)
+      (effects (font (size 1.27 1.27)) hide)
+    )
